File: VER_2/Kicad_project/wzmacniacz_v2.sch (KiCad schematic (older format))
At the start: 65 parts, among them J1 Conn_01x03_Male, J2 AudioJack2_Ground_Switch, J3 AudioJack2_Ground_Switch, SW1 POWER, SW2 STANDBY, SW3 SW_DPDT_x2, T1 Transformer_1P_2S, T2 Transformer_1P_1S, U1 ECC83, U2 EL84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

Commit message: Signed-off-by: unknown <tomasz@fortec.pl>
Parts:
- removed unit 3 of U3
- removed U4: ECC83, Valve:Valve_Noval_P, symbol Valve:ECC83
- added U4: ECC83, Valve:Valve_Noval_P, symbol Valve:ECC83
Connections:
- net at C6.1, R7.2, R9.2: now also U4.1 (A); no longer U1.1 (A)
- net at U1.2 (G): now also LEAD1.2; no longer SW3.2 (B)
- net at C4.1, R6.1: now also U4.3 (K); no longer U1.3 (K)
- net at LA1.2 (+), T1.5 (SC), U1.4 (F1)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: now also U4.4 (F1), U4.5 (F1)
- net at LA1.1 (-), T1.6 (SD), U1.9 (F2)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: now also U4.9 (F2)
- net at U3.7 (G): now also R21.2, R22.2; no longer LEAD1.2
- net at C13.1, R19.2: now also U1.1 (A); no longer U3.6 (A)
- net at C3.1, R18.1: now also U1.3 (K); no longer U3.8 (K)
- net at C14.1, R24.2: now also U3.6 (A)
- net at R23.1: now also U3.8 (K)
- new net: SW3.2 (B), U4.2 (G)
Other:
- moved on the sheet: U1B, U3A
Changed lines of the file:
@@
 L Valve:ECC83 U1
 U 2 1 62E2AB47
-P 2550 4100
-F 0 "U1" H 2778 4146 50  0000 L CNN
-F 1 "ECC83" H 2778 4055 50  0000 L CNN
-F 2 "Valve:Valve_Noval_P" H 2820 3700 50  0001 C CNN
-F 3 "http://www.r-type.org/pdfs/ecc83.pdf" H 2550 4100 50  0001 C CNN
-	2    2550 4100
+P 4800 1850
+F 0 "U1" H 5028 1896 50  0000 L CNN
+F 1 "ECC83" H 5028 1805 50  0000 L CNN
+F 2 "Valve:Valve_Noval_P" H 5070 1450 50  0001 C CNN
+F 3 "http://www.r-type.org/pdfs/ecc83.pdf" H 4800 1850 50  0001 C CNN
+	2    4800 1850
 	1    0    0    -1
 $EndComp
@@
 	7750 3850 8100 3850
 Connection ~ 4100 3450
-$Comp
-L Valve:ECC83 U3
-U 3 1 63FB62E0
-P 3900 7400
-F 0 "U3" H 3672 7271 50  0000 R CNN
-F 1 "ECC83" H 3672 7362 50  0000 R CNN
-F 2 "Valve:Valve_Noval_P" H 4170 7000 50  0001 C CNN
-F 3 "http://www.r-type.org/pdfs/ecc83.pdf" H 3900 7400 50  0001 C CNN
-	3    3900 7400
-	-1   0    0    1
-$EndComp
 Wire Wire Line
 	4000 6500 4400 6500
@@
 $EndComp
 $Comp
-L Valve:ECC83 U4
-U 1 1 64110B5B
-P 6450 1850
-F 0 "U4" H 6678 1896 50  0000 L CNN
-F 1 "ECC83" H 6678 1805 50  0000 L CNN
-F 2 "Valve:Valve_Noval_P" H 6720 1450 50  0001 C CNN
-F 3 "http://www.r-type.org/pdfs/ecc83.pdf" H 6450 1850 50  0001 C CNN
-	1    6450 1850
-	1    0    0    -1
-$EndComp
-$Comp
 L power:GND #PWR020
 U 1 1 64110B55
@@
 L Valve:ECC83 U3
 U 1 1 640605C8
-P 4800 1850
-F 0 "U3" H 5028 1896 50  0000 L CNN
-F 1 "ECC83" H 5028 1805 50  0000 L CNN
-F 2 "Valve:Valve_Noval_P" H 5070 1450 50  0001 C CNN
-F 3 "http://www.r-type.org/pdfs/ecc83.pdf" H 4800 1850 50  0001 C CNN
-	1    4800 1850
+P 6450 1850
+F 0 "U3" H 6678 1896 50  0000 L CNN
+F 1 "ECC83" H 6678 1805 50  0000 L CNN
+F 2 "Valve:Valve_Noval_P" H 6720 1450 50  0001 C CNN
+F 3 "http://www.r-type.org/pdfs/ecc83.pdf" H 6450 1850 50  0001 C CNN
+	1    6450 1850
 	1    0    0    -1
 $EndComp
@@
 	1650 1850 1550 1850
 Connection ~ 1550 1850
+$Comp
+L Valve:ECC83 U4
+U 2 1 63FF4519
+P 2550 4100
+F 0 "U4" H 2778 4146 50  0000 L CNN
+F 1 "ECC83" H 2778 4055 50  0000 L CNN
+F 2 "Valve:Valve_Noval_P" H 2820 3700 50  0001 C CNN
+F 3 "http://www.r-type.org/pdfs/ecc83.pdf" H 2550 4100 50  0001 C CNN
+	2    2550 4100
+	1    0    0    -1
+$EndComp
+$Comp
+L Valve:ECC83 U4
+U 3 1 63FFE0DD
+P 3900 7400
+F 0 "U4" H 3672 7271 50  0000 R CNN
+F 1 "ECC83" H 3672 7362 50  0000 R CNN
+F 2 "Valve:Valve_Noval_P" H 4170 7000 50  0001 C CNN
+F 3 "http://www.r-type.org/pdfs/ecc83.pdf" H 3900 7400 50  0001 C CNN
+	3    3900 7400
+	-1   0    0    1
+$EndComp
 $EndSCHEMATC
